Commit message: update urdf

File: hexapod_description/urdf/hexapod_model.xacro (robot description, xacro)
@@ -121,4 +121,20 @@
         </inertial>
     </link>
+    <joint name="tilt_joint" type="revolute">
+		<parent link="pan_link"/>
+		<child link="tilt_link"/>
+		<axis xyz="0.0 1.0 0.0" />
+		<origin xyz="0.0 0.0 0.020" />
+		<limit lower="-${3.14}" upper="${3.14}" effort="10000" velocity="100" />
+	</joint>
+	<link name="tilt_link">
+        <inertial>
+            <origin xyz="0.0 0.0 0.0" rpy="0.0 0.0 0.0" />
+            <mass value="0.00001"/>
+            <inertia
+                ixx="1.0" ixy="0.0"  ixz="0.0"
+                iyy="1.0" iyz="0.0"
+                izz="1.0" />
+        </inertial>
     <!-- Leg macro -->
     <xacro:macro name="leg" params="side position x y angle axis">

Commit message: upd

File: hexapod_description/urdf/hexapod_model.xacro (robot description, xacro)
@@ -137,4 +137,5 @@
                 izz="1.0" />
         </inertial>
+    </link>
     <!-- Leg macro -->
     <xacro:macro name="leg" params="side position x y angle axis">

Commit message: upd

File: hexapod_description/urdf/hexapod_model.xacro (robot description, xacro)
@@ -124,8 +124,8 @@
 		<parent link="pan_link"/>
 		<child link="tilt_link"/>
-		<axis xyz="0.0 1.0 0.0" />
+		<axis xyz="0.0 1.0 0.0" rpy="0.0 0.0 0.0"/>
 		<origin xyz="0.0 0.0 0.020" />
-		<limit lower="-${3.14}" upper="${3.14}" effort="10000" velocity="100" />
-	</joint>
+		<limit lower="${joint_lower_limit}" upper="${joint_upper_limit}" effort="${joint_effort}" velocity="${joint_velocity}"/>
+    </joint>
 	<link name="tilt_link">
         <inertial>

Commit message: upd

File: hexapod_description/urdf/hexapod_model.xacro (robot description, xacro)
@@ -124,6 +124,6 @@
 		<parent link="pan_link"/>
 		<child link="tilt_link"/>
-		<axis xyz="0.0 1.0 0.0" rpy="0.0 0.0 0.0"/>
-		<origin xyz="0.0 0.0 0.020" />
+		<origin xyz="0.1 0.0 0.034" rpy="0.0 0.0 0.0"/>
+        <axis xyz="0.0 0.0 1.0"/>
 		<limit lower="${joint_lower_limit}" upper="${joint_upper_limit}" effort="${joint_effort}" velocity="${joint_velocity}"/>
     </joint>

Commit message: udpate

File: hexapod_description/urdf/hexapod_model.xacro (robot description, xacro)
@@ -107,5 +107,5 @@
         <parent link="body_link"/>
         <child link="pan_link"/>
-        <origin xyz="0.1 0.0 0.034" rpy="0.0 0.0 0.0"/>
+        <origin xyz="0.0 0.0 0.034" rpy="0.0 0.0 0.0"/>
         <axis xyz="0.0 0.0 1.0"/>
         <limit lower="${joint_lower_limit}" upper="${joint_upper_limit}" effort="${joint_effort}" velocity="${joint_velocity}"/>
@@ -125,5 +125,5 @@
 		<child link="tilt_link"/>
 		<origin xyz="0.1 0.0 0.034" rpy="0.0 0.0 0.0"/>
-        <axis xyz="0.0 0.0 1.0"/>
+        <axis xyz="0.0 0.0 2.0"/>
 		<limit lower="${joint_lower_limit}" upper="${joint_upper_limit}" effort="${joint_effort}" velocity="${joint_velocity}"/>
     </joint>

Commit message: udpate

File: hexapod_description/urdf/hexapod_model.xacro (robot description, xacro)
@@ -124,6 +124,6 @@
 		<parent link="pan_link"/>
 		<child link="tilt_link"/>
-		<origin xyz="0.1 0.0 0.034" rpy="0.0 0.0 0.0"/>
-        <axis xyz="0.0 0.0 2.0"/>
+		<origin xyz="0.0 0.0 0.034" rpy="0.0 0.0 0.0"/>
+        <axis xyz="0.0 0.0 1.0"/>
 		<limit lower="${joint_lower_limit}" upper="${joint_upper_limit}" effort="${joint_effort}" velocity="${joint_velocity}"/>
     </joint>

Commit message: as

File: hexapod_description/urdf/hexapod_model.xacro (robot description, xacro)
@@ -8,5 +8,5 @@
     <xacro:property name="femur_length" value="0.10798"/>
     <xacro:property name="tibia_length" value="0.08774"/>
-    <xacro:property name="tarsus_length" value="0.12065"/>
+    <!-- <xacro:property name="tarsus_length" value="0.12065"/> -->
     <gazebo>
         <plugin name="gazebo_ros_control" filename="libgazebo_ros_control.so">
@@ -52,5 +52,5 @@
     </gazebo>
     <!-- Camera properties -->
-    <joint name="camera_rgb_joint" type="fixed">
+    <!-- <joint name="camera_rgb_joint" type="fixed">
         <parent link="body_link"/>
         <child link="camera_rgb_optical_frame"/>
@@ -81,5 +81,5 @@
                 izz="1.0" />
         </inertial>
-    </link>
+    </link> -->
     <!-- IMU properties -->
     <joint name="imu_joint" type="fixed">
@@ -301,5 +301,5 @@
         </gazebo>
         <!-- tarsus -->
-        <joint name="tarsus_joint_${side}${position}" type="revolute">
+        <!-- <joint name="tarsus_joint_${side}${position}" type="revolute">
             <origin xyz="${tibia_length} 0.0 0.0" rpy="0.0 0.0 0.0"/>
             <parent link="tibia_${side}${position}"/>
@@ -348,9 +348,9 @@
         <gazebo reference="tarsus_${side}${position}">
             <material>Gazebo/DarkGrey</material>
-        </gazebo>
+        </gazebo> -->
         <!-- foot -->
         <joint name="foot_joint_${side}${position}" type="fixed">
-            <origin xyz="${tarsus_length} 0.0 0.0" rpy="0.0 0.0 0.0" />
-            <parent link="tarsus_${side}${position}" />
+            <origin xyz="${tibia_length} 0.0 0.0" rpy="0.0 0.0 0.0" />
+            <parent link="tibia__${side}${position}" />
             <child link="foot_${side}${position}" />
         </joint>

Commit message: as

File: hexapod_description/urdf/hexapod_model.xacro (robot description, xacro)
@@ -8,5 +8,5 @@
     <xacro:property name="femur_length" value="0.10798"/>
     <xacro:property name="tibia_length" value="0.08774"/>
-    <!-- <xacro:property name="tarsus_length" value="0.12065"/> -->
+    <xacro:property name="tarsus_length" value="0.12065"/>
     <gazebo>
         <plugin name="gazebo_ros_control" filename="libgazebo_ros_control.so">
@@ -301,5 +301,5 @@
         </gazebo>
         <!-- tarsus -->
-        <!-- <joint name="tarsus_joint_${side}${position}" type="revolute">
+        <joint name="tarsus_joint_${side}${position}" type="revolute">
             <origin xyz="${tibia_length} 0.0 0.0" rpy="0.0 0.0 0.0"/>
             <parent link="tibia_${side}${position}"/>
@@ -348,9 +348,9 @@
         <gazebo reference="tarsus_${side}${position}">
             <material>Gazebo/DarkGrey</material>
-        </gazebo> -->
+        </gazebo>
         <!-- foot -->
         <joint name="foot_joint_${side}${position}" type="fixed">
-            <origin xyz="${tibia_length} 0.0 0.0" rpy="0.0 0.0 0.0" />
-            <parent link="tibia__${side}${position}" />
+            <origin xyz="${tarsus_length} 0.0 0.0" rpy="0.0 0.0 0.0" />
+            <parent link="tarsus_${side}${position}" />
             <child link="foot_${side}${position}" />
         </joint>

Commit message: as

File: hexapod_description/urdf/hexapod_model.xacro (robot description, xacro)
@@ -52,5 +52,5 @@
     </gazebo>
     <!-- Camera properties -->
-    <!-- <joint name="camera_rgb_joint" type="fixed">
+    <joint name="camera_rgb_joint" type="fixed">
         <parent link="body_link"/>
         <child link="camera_rgb_optical_frame"/>
@@ -81,5 +81,5 @@
                 izz="1.0" />
         </inertial>
-    </link> -->
+    </link>
     <!-- IMU properties -->
     <joint name="imu_joint" type="fixed">
