Commit message: as

File: hexapod_description/urdf/ancabot_model.xacro (robot description, xacro)
@@ -72,5 +72,5 @@
         <origin xyz="0.150 -0.0225 0.034" rpy="${pi/2} ${pi} ${pi/2}"/>
     </joint>
-    <link name="camera_depth_optical_frame">
+    <link name="laser">
         <inertial>
             <origin xyz="0.0 0.0 0.0" rpy="0.0 0.0 0.0" />

Commit message: as

File: hexapod_description/urdf/ancabot_model.xacro (robot description, xacro)
@@ -70,5 +70,5 @@
         <parent link="body_link"/>
         <child link="laser"/>
-        <origin xyz="0.150 -0.0225 0.034" rpy="${pi/2} ${pi} ${pi/2}"/>
+        <origin xyz="0 0 0" rpy="${pi/2} ${pi} ${pi/2}"/>
     </joint>
     <link name="laser">
@@ -86,9 +86,9 @@
         <parent link="body_link"/>
         <child link="imu"/>
-        <origin xyz="0.0 0.0 0.034" rpy="0.0 0.0 0.0"/>
+        <origin xyz="0.0 0.0 0" rpy="0.0 0.0 0.0"/>
     </joint>
     <link name="imu">
         <inertial>
-            <origin xyz="0.0 0.06 0.02" rpy="0.0 0.0 0.0" />
+            <origin xyz="0.0 0 0.0" rpy="0.0 0.0 0.0" />
             <mass value="0.00001"/>
             <inertia

Commit message: as

File: hexapod_description/urdf/ancabot_model.xacro (robot description, xacro)
@@ -74,5 +74,5 @@
     <link name="laser">
         <inertial>
-            <origin xyz="0.0 0.0 0.0" rpy="0.0 0.0 0.0" />
+            <origin xyz="0.06 0.0 0.08" rpy="0.0 0.0 0.0" />
             <mass value="0.00001"/>
             <inertia
@@ -86,9 +86,9 @@
         <parent link="body_link"/>
         <child link="imu"/>
-        <origin xyz="0.0 0.0 0" rpy="0.0 0.0 0.0"/>
+        <origin xyz="0.0 0.0 0.034" rpy="0.0 0.0 0.0"/>
     </joint>
     <link name="imu">
         <inertial>
-            <origin xyz="0.0 0 0.0" rpy="0.0 0.0 0.0" />
+            <origin xyz="0.0 0 0.34" rpy="0.0 0.0 0.0" />
             <mass value="0.00001"/>
             <inertia

Commit message: as

File: hexapod_description/urdf/ancabot_model.xacro (robot description, xacro)
@@ -67,4 +67,5 @@
         </inertial>
     </link> -->
+<!--
     <joint name="laser_joint" type="fixed">
         <parent link="body_link"/>
@@ -81,7 +82,7 @@
                 izz="1.0" />
         </inertial>
-    </link>
+    </link> -->
     <!-- IMU properties -->
-    <joint name="imu_joint" type="fixed">
+    <!-- <joint name="imu_joint" type="fixed">
         <parent link="body_link"/>
         <child link="imu"/>
@@ -97,5 +98,5 @@
                 izz="1.0" />
         </inertial>
-    </link>
+    </link> -->
     <!-- Joint properties -->
     <xacro:property name="joint_lower_limit" value="-${3.14}"/>
